File: Tamagotchi/Tamagotchi.kicad_sch (KiCad schematic)
At the start: 78 parts, among them J1 CH_USB_C, J2 display: GMT085-01, J3 JTAG, Q1 ZVP1320FTA, Q2 SS8050-MS, SW1 A, SW2 B, SW3 C, SW4 BOOT, SW5 NRST, U1 MCP73833, U2 STM32U031K4Ux, U3 AT25EU0021A-MAHN-T, U4 AP7343D-33W5, Y1 32.786KHz

Commit message: Fixed power section
Parts:
- removed C14: 100n, Capacitor_SMD:C_0603_1608Metric, symbol Device:C_Small
- removed J2: display: GMT085-01, Marijn:GMT085-01, symbol Connector_Generic:Conn_01x12
- removed Q2: SS8050-MS, Package_TO_SOT_SMD:SOT-23, symbol Transistor_BJT:SS8050
- removed R10: 5R1, Resistor_SMD:R_0603_1608Metric, symbol Device:R_Small
- removed R19: 10k, Resistor_SMD:R_0603_1608Metric, symbol Device:R_Small
- removed R20: 51k, Resistor_SMD:R_0603_1608Metric, symbol Device:R_Small
- added C16, C6: 1u, Capacitor_SMD:C_0603_1608Metric, symbol Device:C_Small
- added C17: 4u7, Capacitor_SMD:C_0603_1608Metric, symbol Device:C_Small
- added C18: 100n, Capacitor_SMD:C_0603_1608Metric, symbol Device:C_Small
- added C5: 4u7, PCM_Capacitor_Tantalum_SMD_AKL:CP_EIA-3216-18_Kemet-A, symbol Device:C_Small
- added D5: USL1G, Diode_SMD:D_SOD-123F, symbol Device:D_Small
- added J2: OLED_FB, Connector_PinHeader_2.54mm:PinHeader_1x07_P2.54mm_Vertical, symbol Connector_Generic:Conn_01x07
- added J3: FFC2B35-30-T, Marijn:FFC2B35-30, symbol Connector_Generic:Conn_01x30
- added R18: 560k, Resistor_SMD:R_0603_1608Metric, symbol Device:R_Small
- added TP1: SWCLK, TestPoint:TestPoint_Pad_D1.5mm, symbol Connector:TestPoint
- added TP2: SWDIO, TestPoint:TestPoint_Pad_D1.5mm, symbol Connector:TestPoint
- added TP3: GND, TestPoint:TestPoint_Pad_D1.5mm, symbol Connector:TestPoint
- added TP4: 3v3, TestPoint:TestPoint_Pad_D1.5mm, symbol Connector:TestPoint
- C3: value 100n -> 10u
- R6: renamed from R7; value 10k -> 2k
- R9: value 2k2 -> 50r
- renumbered C8 to C10, C9 to C11, C10 to C12, C11 to C13, C12 to C14, C13 to C15, C15 to C19, C16 to C20, C17 to C21, C18 to C22, C19 to C23, C5 to C7, C6 to C8, C7 to C9, D9 to D10, D10 to D11, D11 to D12, D12 to D13, D13 to D14, D5 to D6, D6 to D7, D7 to D8, D8 to D9, J3 to J4, R2 to R1, R11 to R10, R12 to R11, R13 to R12, R14 to R13, R15 to R14, R16 to R15, R17 to R16, R18 to R17, R21 to R19, R1 to R2, R22 to R20, R23 to R21, R24 to R22, R5 to R4, R6 to R5, R4 to R7, TP1 to TP5, TP2 to TP6
Connections:
- net +3V3: now also C3.2, C4.2, C17.1, C18.1, C6.1, J2.7 (Pin_7), J3.2 (Pin_2), J3.27 (Pin_27), J3.4 (Pin_4), TP4.1; no longer C3.1, C4.1
- net GND: now also C3.1, C4.1, C16.2, C17.2, C18.2, C5.2, C6.2, D5.1 (K), J2.6 (Pin_6), J3.1 (Pin_1), J3.10 (Pin_10), J3.11 (Pin_11), J3.15 (Pin_15), J3.16 (Pin_16), J3.17 (Pin_17), J3.18 (Pin_18), J3.28 (Pin_28), J3.30 (Pin_30), J3.7 (Pin_7), J3.8 (Pin_8), J3.9 (Pin_9), R18.2, TP3.1; no longer C3.2, C4.2
- net SWCLK: now also TP1.1
- net SWDIO: now also TP2.1
- net OLED_VSL: now reaches R9.1
- net OLED_VSL: now also J3.5 (Pin_5)
- net TFT_BL: no longer names the net of R9.2
- net TFT_BL: now also D5.2 (A); no longer U2.27 (PB4)
- net TFT_DC renamed OLED_DC
- net OLED_DC: now also J2.3 (Pin_3), J3.20 (Pin_20)
- net TFT_NRST renamed OLED_NRST
- net OLED_NRST: now also J2.1 (Pin_1), J3.21 (Pin_21)
- net TFT_SPI_MOSI renamed OLED_SPI_MOSI
- net OLED_SPI_MOSI: now also J2.4 (Pin_4), J3.13 (Pin_13)
- net TFT_SPI_NSS renamed OLED_SPI_NSS
- net OLED_SPI_NSS: now also J2.2 (Pin_2), J3.19 (Pin_19)
- net TFT_SPI_SCK renamed OLED_SPI_SCK
- net OLED_SPI_SCK: now also J2.5 (Pin_5), J3.14 (Pin_14)
- new net: C16.1, J3.26 (Pin_26)
- new net: C5.1, J3.3 (Pin_3)
- new net OLED_IREF: J3.22 (Pin_22), R18.1
- no-connect marks 11 -> 18
Other:
- note added: "1,5 inch OLED-schermmodule SPI 7Pin 128*128"
- note added: "500mA"
- note added: "6800/8080 mode signals and BS0/1 = 0 for 3/4 wire SPI"
- note added: "D2 = NC for 3/4 wire SPI"
- note added: "D3-D7 = 0 (VSS)"
- note added: "DISPLAY: NHD-1.5-128128G"
- note added: "Display"
- note removed: "100mA"
- note removed: "TFT"
- moved on the sheet: BT1, C1, C2, D1, D2, D3, D4, F1, J1, R1, R3, R4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

Commit message: Removed old note
Other:
- note removed: "DISPLAY: https://nl.aliexpress.com/item/1005005039754957.html?spm=a2g0o.productlist.main.28.6ceaFg0hFg0hn5&algo_pvid=c510dd45-5260-4aa8-843d-e0720577f99c&algo_exp_id=c510dd45-5260-4aa8-843d-e0720577f99c-31&pdp_ext_f=%7B%22order%22%3A%22-1%22%2C%22eval%22%3A%221%22%7D&pdp_npi=6%40dis%21EUR%212.53%212.07%21%21%212.88%212.36%21%402103892f17553668013963929e3f58%2112000031419530217%21sea%21NL%210%21AB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"
Changed lines of the file:
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@@
-		)
-	)
-	(text "DISPLAY: https://nl.aliexpress.com/item/1005005039754957.html?spm=a2g0o.productlist.main.28.6ceaFg0hFg0hn5&algo_pvid=c510dd45-5260-4aa8-843d-e0720577f99c&algo_exp_id=c510dd45-5260-4aa8-843d-e0720577f99c-31&pdp_ext_f=%7B%22order%22%3A%22-1%22%2C%22eval%22%3A%221%22%7D&pdp_npi=6%40dis%21EUR%212.53%212.07%21%21%212.88%212.36%21%402103892f17553668013963929e3f58%2112000031419530217%21sea%21NL%210%21ABX%211%210%21n_tag%3A-29910%3Bm03_new_user%3A-29895&curPageLogUid=YYKFiAIGsFCS&utparam-url=scene%3Asearch%7Cquery_from%3A%7Cx_object_id%3A1005005039754957%7C_p_origin_prod%3A&_gl=1*lcgtoe*_gcl_aw*R0NMLjE3NTUzNjY3ODIuQ2owS0NRancySURGQmhEQ0FSSXNBQkRLT0o1QllkU0RhUVh5T2EzdXE4TjF1aE1iMkZDUldlV2w5dmZhNTAzWEtrSUtWYUhRNWQxVWl1QWFBcm9PRUFMd193Y0I.*_gcl_dc*R0NMLjE3NTUzNjY3ODIuQ2owS0NRancySURGQmhEQ0FSSXNBQkRLT0o1QllkU0RhUVh5T2EzdXE4TjF1aE1iMkZDUldlV2w5dmZhNTAzWEtrSUtWYUhRNWQxVWl1QWFBcm9PRUFMd193Y0I.*_gcl_au*ODc3MDc2NjQ0LjE3NTUwMDc5MjY.*_ga*MjE4NTczNTYuMTc1NTAwNzkyNg..*_ga_VED1YSGNC7*czE3NTUzNjY3ODEkbzMkZzEkdDE3NTUzNjY4MDYkajM1JGwwJGgw"
-		(exclude_from_sim no)
-		(at 229.616 225.552 0)
-		(effects
-			(font
-				(size 1.27 1.27)
-			)
 		)
 	)
